File: Console/A/airboy.kicad_sch (KiCad schematic)
At the start: 25 parts, among them J1 cartridge port, J2 display connector, J8 touch, Q1 MMBT3906, U1 eeprom

Commit message: info changes
Other:
- company: (none) -> AirBoy Company (Piotr Mijakowski)
- title: (none) -> AirBoy
Changed lines of the file:
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@@
 (kicad_sch (version 20211123) (generator eeschema)
   (paper "A4")
+  (title_block
+    (title "AirBoy")
+    (date "2023-03-31")
+    (rev "2.1A")
+    (company "AirBoy Company (Piotr Mijakowski)")
+  )
   (junction (at 41.91 175.26) (diameter 0) (color 0 0 0 0)
   )
