File: Console/A/audio.kicad_sch (KiCad schematic)
At the start: 55 parts, among them J3 SPK right, J4 SPK left, J5 AudioJack, U6 PCM5100A, U7 LM4936

Commit message: info changes
Other:
- company: (none) -> AirBoy Company (Piotr Mijakowski)
- title: (none) -> AirBoy - Audio
Changed lines of the file:
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@@
 (kicad_sch (version 20211123) (generator eeschema)
   (paper "A4")
+  (title_block
+    (title "AirBoy - Audio")
+    (date "2023-03-31")
+    (rev "2.1A")
+    (company "AirBoy Company (Piotr Mijakowski)")
+  )
   (junction (at 67.31 134.62) (diameter 0) (color 0 0 0 0)
   )
