File: Console/A/microcontroller.kicad_sch (KiCad schematic)
At the start: 32 parts, among them SW1 SW_BOOT, SW2 SW_RST, U2 ESP32-S3, Y1 40 Mhz

Commit message: info changes
Other:
- company: (none) -> AirBoy Company (Piotr Mijakowski)
- title: (none) -> AirBoy - Microcontroler
Changed lines of the file:
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@@
 (kicad_sch (version 20211123) (generator eeschema)
   (paper "A4")
+  (title_block
+    (title "AirBoy - Microcontroler")
+    (date "2023-03-31")
+    (rev "2.1A")
+    (company "AirBoy Company (Piotr Mijakowski)")
+  )
   (junction (at 86.36 158.75) (diameter 0) (color 0 0 0 0)
   )
