File: Console/A/power.kicad_sch (KiCad schematic)
At the start: 36 parts, among them J6 USBC, J7 JST, SW16 PW_SWICH, U10 AP7362A, U8 BQ24075RGT, U9 USBLC6-2SC6

Commit message: info changes
Other:
- note added: "Do not buy BQ24075T version"
- company: (none) -> AirBoy Company (Piotr Mijakowski)
- title: (none) -> AirBoy - Power
Changed lines of the file:
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@@
 (kicad_sch (version 20211123) (generator eeschema)
   (paper "A4")
+  (title_block
+    (title "AirBoy - Power")
+    (date "2023-03-31")
+    (rev "2.1A")
+    (company "AirBoy Company (Piotr Mijakowski)")
+  )
   (junction (at 104.14 36.83) (diameter 0) (color 0 0 0 0)
   )
@@
     (effects (font (size 1.27 1.27)) (justify left bottom))
   )
+  (text "Do not buy BQ24075T version" (at 85.09 149.86 0)
+    (effects (font (size 1.27 1.27)) (justify left bottom))
+  )
