File: Console/A/controller.kicad_sch (KiCad schematic)
At the start: 31 parts, among them SW10 SW_Y, SW11 SW_X, SW12 SW_LTRIG, SW13 SW_AIRBOY, SW14 SW_SELECT, SW15 SW_START, SW3 SW UP, SW4 SW_DOWN, SW5 SW_LEFT, SW6 SW_RIGHT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

Commit message: info changes
Other:
- company: (none) -> AirBoy Company (Piotr Mijakowski)
- title: (none) -> AirBoy - Controler
Changed lines of the file:
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@@
 (kicad_sch (version 20211123) (generator eeschema)
   (paper "A4")
+  (title_block
+    (title "AirBoy - Controler")
+    (date "2023-03-31")
+    (rev "2.1A")
+    (company "AirBoy Company (Piotr Mijakowski)")
+  )
   (junction (at 255.27 55.88) (diameter 0) (color 0 0 0 0)
   )

Commit message: modified PCB and output gerber files
Connections:
- net GND: now also SW7. (B), SW7.2 (B); no longer SW12.2 (A), SW7.3 (B), SW7.4 (B)
- net at C24.1, R21.2: now also SW12.2 (B); no longer SW12.3 (B), SW12.4 (B)
- net at C23.1, R20.2, SW7.1 (A): no longer SW7.2 (A)
Changed lines of the file:
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@@
   (junction (at 152.4 68.58) (diameter 0) (color 0 0 0 0)
   )
+  (junction (at 198.12 129.54) (diameter 0) (color 0 0 0 0)
+  )
   (junction (at 255.27 76.2) (diameter 0) (color 0 0 0 0)
   )
@@
   (junction (at 167.64 85.09) (diameter 0) (color 0 0 0 0)
   )
+  (junction (at 200.66 129.54) (diameter 0) (color 0 0 0 0)
+  )
   (junction (at 152.4 53.34) (diameter 0) (color 0 0 0 0)
   )
@@
     (stroke (width 0) (type default) (color 0 0 0 0))
   )
+  (wire (pts (xy 198.12 127) (xy 198.12 129.54))
+    (stroke (width 0) (type default) (color 0 0 0 0))
+  )
   (wire (pts (xy 137.16 176.53) (xy 139.7 176.53))
     (stroke (width 0) (type default) (color 0 0 0 0))
@@
     (stroke (width 0) (type default) (color 0 0 0 0))
   )
+  (wire (pts (xy 198.12 129.54) (xy 200.66 129.54))
+    (stroke (width 0) (type default) (color 0 0 0 0))
+  )
   (wire (pts (xy 240.03 55.88) (xy 240.03 53.34))
     (stroke (width 0) (type default) (color 0 0 0 0))
@@
     (stroke (width 0) (type default) (color 0 0 0 0))
   )
-  (wire (pts (xy 200.66 124.46) (xy 200.66 137.16))
+  (wire (pts (xy 200.66 124.46) (xy 200.66 129.54))
+    (stroke (width 0) (type default) (color 0 0 0 0))
+  )
+  (wire (pts (xy 200.66 129.54) (xy 200.66 137.16))
     (stroke (width 0) (type default) (color 0 0 0 0))
   )
@@
     (stroke (width 0) (type default) (color 0 0 0 0))
   )
+  (wire (pts (xy 252.73 124.46) (xy 252.73 137.16))
+    (stroke (width 0) (type default) (color 0 0 0 0))
+  )
   (wire (pts (xy 57.15 140.97) (xy 69.85 140.97))
     (stroke (width 0) (type default) (color 0 0 0 0))
@@
     (stroke (width 0) (type default) (color 0 0 0 0))
   )
-  (wire (pts (xy 252.73 124.46) (xy 252.73 137.16))
-    (stroke (width 0) (type default) (color 0 0 0 0))
-  )
   (wire (pts (xy 87.63 119.38) (xy 87.63 121.92))
     (stroke (width 0) (type default) (color 0 0 0 0))
@@
     (stroke (width 0) (type default) (color 0 0 0 0))
   )
+  (wire (pts (xy 187.96 127) (xy 187.96 129.54))
+    (stroke (width 0) (type default) (color 0 0 0 0))
+  )
   (wire (pts (xy 95.25 130.81) (xy 106.68 130.81))
     (stroke (width 0) (type default) (color 0 0 0 0))
@@
   )
   (wire (pts (xy 95.25 82.55) (xy 106.68 82.55))
+    (stroke (width 0) (type default) (color 0 0 0 0))
+  )
+  (wire (pts (xy 187.96 129.54) (xy 198.12 129.54))
     (stroke (width 0) (type default) (color 0 0 0 0))
   )
@@
   (symbol (lib_id "Device:C") (at 236.22 130.81 0) (unit 1)
     (in_bom yes) (on_board yes)
-    (property "Reference" "C24" (id 0) (at 238.76 129.54 0)
-      (effects (font (size 1.27 1.27)) (justify left))
-    )
-    (property "Value" "100n" (id 1) (at 238.76 132.08 0)
+    (property "Reference" "C24" (id 0) (at 228.6 129.54 0)
+      (effects (font (size 1.27 1.27)) (justify left))
+    )
+    (property "Value" "100n" (id 1) (at 228.6 132.08 0)
       (effects (font (size 1.27 1.27)) (justify left))
     )
@@
     )
     (pin "1")
-    (pin "3")
-    (pin "2")
-    (pin "4")
+    (pin "2")
+    (pin "")
+    (pin "")
   )
   (symbol (lib_id "Switch:SW_MEC_5E") (at 200.66 55.88 0) (unit 1)
@@
     )
     (pin "1")
-    (pin "3")
-    (pin "2")
-    (pin "4")
+    (pin "2")
+    (pin "")
+    (pin "")
   )
   (symbol (lib_id "Device:R") (at 54.61 68.58 0) (unit 1)
@@
   (symbol (lib_id "Device:C") (at 184.15 130.81 0) (unit 1)
     (in_bom yes) (on_board yes)
-    (property "Reference" "C23" (id 0) (at 186.69 129.54 0)
-      (effects (font (size 1.27 1.27)) (justify left))
-    )
-    (property "Value" "100n" (id 1) (at 186.69 132.08 0)
-      (effects (font (size 1.27 1.27)) (justify left))
-    )
+    (property "Reference" "C23" (id 0) (at 176.53 129.54 0)
+      (effects (font (size 1.27 1.27)) (justify left))
+    )
+    (property "Value" "100n" (id 1) (at 176.53 132.08 0)
+      (effects (font (size 1.27 1.27)) (justify left))
+    )
