File: Cartridge/Dev/A/airboy_cartridge.kicad_pcb (KiCad board)
At the start: 2 copper layers, 51.6 x 35.8 mm, 36 parts, among them J1 USB, J2 Micro_SD_Card, J3 EXT, J4 edge, Q1 S8050, Q2 S8050, U1 CH340G, U2 GD25Q64C, U4 USBLC6-2SC6, Y1 12MHz

Commit message: modified PCB and output gerber files
Changed lines of the file:
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@@
       (layerselection 0x00010fc_ffffffff)
       (disableapertmacros false)
-      (usegerberextensions false)
+      (usegerberextensions true)
       (usegerberattributes true)
       (usegerberadvancedattributes true)
-      (creategerberjobfile true)
+      (creategerberjobfile false)
       (svguseinch false)
       (svgprecision 6)
@@
       (plotinvisibletext false)
       (sketchpadsonfab false)
-      (subtractmaskfromsilk false)
+      (subtractmaskfromsilk true)
       (outputformat 1)
       (mirror false)
-      (drillshape 1)
+      (drillshape 0)
       (scaleselection 1)
-      (outputdirectory "")
+      (outputdirectory "out/")
     )
   )
@@
     (fp_line (start -1.6 0.4) (end -1.6 -0.8) (layer "B.Fab") (width 0.1))
     (fp_line (start -1.6 -0.8) (end 1.6 -0.8) (layer "B.Fab") (width 0.1))
-    (pad "1" smd roundrect (at -1.4375 0 90) (size 1.575 1.35) (layers "B.Cu" "B.Paste" "B.Mask") (roundrect_rratio 0.185185)
+    (pad "1" smd roundrect (at -1.4375 0 90) (size 1.575 1.35) (layers "B.Cu" "B.Paste" "B.Mask") (roundrect_rratio 0.1851851852)
       (net 5 "/VDD_SPI") (pintype "passive"))
-    (pad "2" smd roundrect (at 1.4375 0 90) (size 1.575 1.35) (layers "B.Cu" "B.Paste" "B.Mask") (roundrect_rratio 0.185185)
+    (pad "2" smd roundrect (at 1.4375 0 90) (size 1.575 1.35) (layers "B.Cu" "B.Paste" "B.Mask") (roundrect_rratio 0.1851851852)
       (net 2 "GND") (pintype "passive"))
     (model "${KICAD6_3DMODEL_DIR}/Capacitor_Tantalum_SMD.3dshapes/CP_EIA-3216-18_Kemet-A.wrl"
@@
     (fp_line (start -1.6 -0.8) (end 1.6 -0.8) (layer "B.Fab") (width 0.1))
     (fp_line (start -1.2 0.8) (end -1.6 0.4) (layer "B.Fab") (width 0.1))
-    (pad "1" smd roundrect (at -1.4375 0 180) (size 1.575 1.35) (layers "B.Cu" "B.Paste" "B.Mask") (roundrect_rratio 0.185185)
+    (pad "1" smd roundrect (at -1.4375 0 180) (size 1.575 1.35) (layers "B.Cu" "B.Paste" "B.Mask") (roundrect_rratio 0.1851851852)
       (net 4 "+3.3V") (pintype "passive"))
-    (pad "2" smd roundrect (at 1.4375 0 180) (size 1.575 1.35) (layers "B.Cu" "B.Paste" "B.Mask") (roundrect_rratio 0.185185)
+    (pad "2" smd roundrect (at 1.4375 0 180) (size 1.575 1.35) (layers "B.Cu" "B.Paste" "B.Mask") (roundrect_rratio 0.1851851852)
       (net 2 "GND") (pintype "passive"))
     (model "${KICAD6_3DMODEL_DIR}/Capacitor_Tantalum_SMD.3dshapes/CP_EIA-3216-18_Kemet-A.wrl"
@@
     (fp_line (start 1.6 -0.8) (end 1.6 0.8) (layer "B.Fab") (width 0.1))
     (fp_line (start 1.6 0.8) (end -1.2 0.8) (layer "B.Fab") (width 0.1))
-    (pad "1" smd roundrect (at -1.4375 0 180) (size 1.575 1.35) (layers "B.Cu" "B.Paste" "B.Mask") (roundrect_rratio 0.185185)
+    (pad "1" smd roundrect (at -1.4375 0 180) (size 1.575 1.35) (layers "B.Cu" "B.Paste" "B.Mask") (roundrect_rratio 0.1851851852)
       (net 4 "+3.3V") (pintype "passive"))
-    (pad "2" smd roundrect (at 1.4375 0 180) (size 1.575 1.35) (layers "B.Cu" "B.Paste" "B.Mask") (roundrect_rratio 0.185185)
+    (pad "2" smd roundrect (at 1.4375 0 180) (size 1.575 1.35) (layers "B.Cu" "B.Paste" "B.Mask") (roundrect_rratio 0.1851851852)
       (net 2 "GND") (pintype "passive"))
     (model "${KICAD6_3DMODEL_DIR}/Capacitor_Tantalum_SMD.3dshapes/CP_EIA-3216-18_Kemet-A.wrl"
@@
     (fp_line (start -1.6 0.4) (end -1.6 -0.8) (layer "B.Fab") (width 0.1))
     (fp_line (start -1.2 0.8) (end -1.6 0.4) (layer "B.Fab") (width 0.1))
-    (pad "1" smd roundrect (at -1.4375 0) (size 1.575 1.35) (layers "B.Cu" "B.Paste" "B.Mask") (roundrect_rratio 0.185185)
+    (pad "1" smd roundrect (at -1.4375 0) (size 1.575 1.35) (layers "B.Cu" "B.Paste" "B.Mask") (roundrect_rratio 0.1851851852)
       (net 4 "+3.3V") (pintype "passive"))
-    (pad "2" smd roundrect (at 1.4375 0) (size 1.575 1.35) (layers "B.Cu" "B.Paste" "B.Mask") (roundrect_rratio 0.185185)
+    (pad "2" smd roundrect (at 1.4375 0) (size 1.575 1.35) (layers "B.Cu" "B.Paste" "B.Mask") (roundrect_rratio 0.1851851852)
       (net 2 "GND") (pintype "passive"))
     (model "${KICAD6_3DMODEL_DIR}/Capacitor_Tantalum_SMD.3dshapes/CP_EIA-3216-18_Kemet-A.wrl"
@@
     )
   )
+  (gr_circle (center 139.446 113.03) (end 139.646 113.03) (layer "B.SilkS") (width 0.15) (fill solid))
+  (gr_circle (center 142.494 99.568) (end 142.694 99.568) (layer "B.SilkS") (width 0.15) (fill solid))
+  (gr_circle (center 136.144 99.822) (end 136.344 99.822) (layer "B.SilkS") (width 0.15) (fill solid))
   (gr_line (start 124.2 86) (end 124.2 121.3) (layer "Edge.Cuts") (width 0.1))
   (gr_line (start 175.8 86) (end 175.8 121.3) (layer "Edge.Cuts") (width 0.1))
@@
   (segment (start 169.6974 114.3508) (end 170.9674 114.3508) (width 0.508) (layer "F.Cu") (net 2))
   (segment (start 126.18 88.085) (end 134.82 88.085) (width 0.508) (layer "F.Cu") (net 2))
-  (segment (start 145.555 115.049) (end 145.555 118.6) (width 0.508) (layer "F.Cu") (net 2))
   (segment (start 141.1478 106.1212) (end 141.1478 104.6734) (width 0.508) (layer "F.Cu") (net 2))
   (segment (start 136.1059 96.7359) (end 134.2136 94.8436) (width 0.508) (layer "F.Cu") (net 2))
@@
   (segment (start 132.842 103.632) (end 134.0104 102.4636) (width 0.508) (layer "F.Cu") (net 2))
   (segment (start 165.5826 89.027) (end 165.5826 91.4146) (width 0.508) (layer "F.Cu") (net 2))
+  (segment (start 145.555 118.5) (end 145.555 115.049) (width 0.508) (layer "F.Cu") (net 2))
   (segment (start 169.1894 113.8428) (end 169.1894 112.9792) (width 0.508) (layer "F.Cu") (net 2))
   (segment (start 131.572 111.76) (end 131.572 110.744) (width 0.508) (layer "F.Cu") (net 2))
@@
   (segment (start 146.7866 109.601) (end 145.8468 110.5408) (width 0.1778) (layer "B.Cu") (net 31))
   (segment (start 147.872 109.601) (end 146.7866 109.601) (width 0.1778) (layer "B.Cu") (net 31))
-  (segment (start 146.812 118.587) (end 146.825 118.6) (width 0.1778) (layer "F.Cu") (net 32))
   (segment (start 145.4404 113.6396) (end 146.812 115.0112) (width 0.1778) (layer "F.Cu") (net 32))
   (segment (start 146.812 115.0112) (end 146.812 118.587) (width 0.1778) (layer "F.Cu") (net 32))
